File: debug.kicad_pcb (KiCad board)
At the start: 2 copper layers, 47 parts, among them J1 ZX62D-AB-5P8, P1 LPC-Link, P2 UART, P3 JTAG, P4 Cortex-Debug, P5 Vout, U1 93C46, U2 PRTR5V0U2X, U3 FT2232H, U4 LD1117S33CTR, X1 12MHz

Commit message: place and route in progress...
Parts:
- moved P5 61.4 mm to (90.9, 83.6), turned to 270 degrees
- moved R6 58.1 mm to (91.9, 118.4)
- moved C2 57.6 mm to (91.2, 99.3), turned to 270 degrees
- moved R5 57.4 mm to (91.2, 108.0)
- moved C3 54.0 mm to (98.3, 85.1), turned to 270 degrees
- moved C1 54.0 mm to (95.0, 98.0)
- moved R4 50.5 mm to (99.1, 94.5), turned to 90 degrees
- moved R2 48.3 mm to (101.3, 94.5), turned to 90 degrees
- moved C12 48.0 mm to (102.6, 119.1), turned to 270 degrees
- moved R3 46.1 mm to (103.6, 94.5), turned to 270 degrees
- moved R1 43.9 mm to (105.9, 94.5), turned to 90 degrees
- moved C13 42.7 mm to (108.2, 119.1), turned to 270 degrees
- moved C16 38.8 mm to (111.3, 94.0)
- moved R11 38.5 mm to (111.0, 96.5)
- moved R10 38.1 mm to (111.0, 98.6)
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Routing:
- net Net-(FB1-Pad1): track 0.00 -> 23.2 mm
- net /USB_JTAG_DM: track 0.00 -> 20.0 mm
- net /USB_JTAG_DP: track 0.00 -> 19.5 mm
- net Net-(C7-Pad1): track 20.3 -> 6.91 mm, vias 2 -> 0
- net /FT_XTOUT: track 0.00 -> 11.3 mm
- net Net-(R6-Pad2): track 0.00 -> 11.1 mm
- net /FT_XTIN: track 0.00 -> 9.95 mm
- net Net-(R5-Pad2): track 0.00 -> 6.82 mm
- net Net-(C5-Pad1): track 0.00 -> 6.40 mm
- net Net-(FB3-Pad1): track 0.00 -> 2.70 mm
- net /USB_JTAG_1.8V: track 7.23 -> 9.92 mm
Other:
- board outline added: 56.4 x 42.2 mm
